File: Grad_Cap.kicad_pcb (KiCad board)
At the start: 2 copper layers, 339.4 x 339.4 mm, 88 parts, among them U1 ItsyBitsy 32u4 5V

Commit message: cap + refs gone
Parts:
- added C1: 50u, Capacitor_SMD:C_1206_3216Metric_Pad1.33x1.80mm_HandSolder, F.Cu at (210.5, 211.4)
Routing:
- net GND: track 170.8 -> 172.4 mm, vias 86 -> 87

Commit message: Pads Added
Parts:
- added TP1: TestPoint, TestPoint:TestPoint_Pad_3.0x3.0mm, B.Cu at (215.0, 185.0)
- added TP2: TestPoint, TestPoint:TestPoint_Pad_3.0x3.0mm, B.Cu at (155.0, 185.0)
Routing:
- net +5V: track 0.00 -> 3.71 mm, vias 0 -> 1
Changed lines of the file:
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@@
     )
+  )
+  (footprint "TestPoint:TestPoint_Pad_3.0x3.0mm" (layer "B.Cu")
+    (at 155 185 180)
+    (descr "SMD rectangular pad as test Point, square 3.0mm side length")
+    (tags "test point SMD pad rectangle square")
+    (property "Sheetfile" "Grad_Cap.kicad_sch")
+    (property "Sheetname" "")
+    (attr exclude_from_pos_files)
+    (fp_text reference "TP2" (at 0 2.398) (layer "B.SilkS")
+      (effects (font (size 1 1) (thickness 0.15)) (justify mirror))
+    )
+    (fp_text value "TestPoint" (at 0 -2.55) (layer "B.Fab")
+      (effects (font (size 1 1) (thickness 0.15)) (justify mirror))
+    )
+    (fp_text user "${REFERENCE}" (at 0 2.4) (layer "B.Fab")
+      (effects (font (size 1 1) (thickness 0.15)) (justify mirror))
+    )
+    (fp_line (start 1.7 1.7) (end 1.7 -1.7) (layer "B.SilkS") (width 0.12))
+    (fp_line (start -1.7 -1.7) (end -1.7 1.7) (layer "B.SilkS") (width 0.12))
+    (fp_line (start 1.7 -1.7) (end -1.7 -1.7) (layer "B.SilkS") (width 0.12))
+    (fp_line (start -1.7 1.7) (end 1.7 1.7) (layer "B.SilkS") (width 0.12))
+    (fp_line (start -2 2) (end 2 2) (layer "B.CrtYd") (width 0.05))
+    (fp_line (start 2 -2) (end 2 2) (layer "B.CrtYd") (width 0.05))
+    (fp_line (start 2 -2) (end -2 -2) (layer "B.CrtYd") (width 0.05))
+    (fp_line (start -2 2) (end -2 -2) (layer "B.CrtYd") (width 0.05))
+    (pad "1" smd rect (at 0 0 180) (size 3 3) (layers "B.Cu" "B.Mask")
+      (net 1 "GND") (pinfunction "1") (pintype "passive"))
+  )
+  (footprint "TestPoint:TestPoint_Pad_3.0x3.0mm" (layer "B.Cu")
+    (at 215 185 180)
+    (descr "SMD rectangular pad as test Point, square 3.0mm side length")
+    (tags "test point SMD pad rectangle square")
+    (property "Sheetfile" "Grad_Cap.kicad_sch")
+    (property "Sheetname" "")
+    (attr exclude_from_pos_files)
+    (fp_text reference "TP1" (at 0 2.398) (layer "B.SilkS")
+      (effects (font (size 1 1) (thickness 0.15)) (justify mirror))
+    )
+    (fp_text value "TestPoint" (at 0 -2.55) (layer "B.Fab")
+      (effects (font (size 1 1) (thickness 0.15)) (justify mirror))
+    )
+    (fp_text user "${REFERENCE}" (at 0 2.4) (layer "B.Fab")
+      (effects (font (size 1 1) (thickness 0.15)) (justify mirror))
+    )
+    (fp_line (start -1.7 -1.7) (end -1.7 1.7) (layer "B.SilkS") (width 0.12))
+    (fp_line (start 1.7 -1.7) (end -1.7 -1.7) (layer "B.SilkS") (width 0.12))
+    (fp_line (start -1.7 1.7) (end 1.7 1.7) (layer "B.SilkS") (width 0.12))
+    (fp_line (start 1.7 1.7) (end 1.7 -1.7) (layer "B.SilkS") (width 0.12))
+    (fp_line (start 2 -2) (end 2 2) (layer "B.CrtYd") (width 0.05))
+    (fp_line (start -2 2) (end -2 -2) (layer "B.CrtYd") (width 0.05))
+    (fp_line (start -2 2) (end 2 2) (layer "B.CrtYd") (width 0.05))
+    (fp_line (start 2 -2) (end -2 -2) (layer "B.CrtYd") (width 0.05))
+    (pad "1" smd rect (at 0 0 180) (size 3 3) (layers "B.Cu" "B.Mask")
+      (net 2 "+5V") (pinfunction "1") (pintype "passive"))
   )
   (gr_circle (center 185 185) (end 196.999999 185) (layer "Edge.Cuts") (width 0.1) (fill none))
@@
   (via (at 231.9528 268.1986) (size 0.8) (drill 0.4) (layers "F.Cu" "B.Cu") (net 1))
   (via (at 198.85 201.0344) (size 0.8) (drill 0.4) (layers "F.Cu" "B.Cu") (net 1))
+  (via (at 211.289 185) (size 1.5) (drill 1) (layers "F.Cu" "B.Cu") (net 2))
+  (segment (start 211.289 185) (end 215 185) (width 2.5) (layer "B.Cu") (net 2))
   (segment (start 222.34 244.3478) (end 222.34 247.7921) (width 0.7) (layer "F.Cu") (net 3))
   (segment (start 222.34 247.7921) (end 227.24 252.6921) (width 0.7) (layer "F.Cu") (net 3))
@@
     (connect_pads (clearance 0.35))
     (min_thickness 0.25) (filled_areas_thickness no)
-    (fill yes (thermal_gap 0.5) (thermal_bridge_width 0.5))
+    (fill yes (thermal_gap 0.5) (thermal_bridge_width 0.7))
     (polygon
       (pts

Commit message: Dip Switch
Parts:
- added SW1: SW_SPST, Button_Switch_SMD:SW_DIP_SPSTx01_Slide_6.7x4.1mm_W6.73mm_P2.54mm_LowProfile_JPin, F.Cu at (211.0, 185.0)
Connections:
- TP1 pad 1: +5V -> Net-(TP1-Pad1)
Routing:
- net Net-(TP1-Pad1): track 0.00 -> 14.5 mm, vias 0 -> 1
- net +5V: track 3.71 -> 0.00 mm, vias 1 -> 0
Changed lines of the file:
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@@
   (net 111 "Net-(D84-Pad4)")
   (net 112 "unconnected-(U1-Pad19)")
+  (net 113 "Net-(TP1-Pad1)")
   (footprint "LED_SMD:LED_Inolux_IN-PI554FCH_PLCC4_5.0x5.0mm_P3.2mm" placed (layer "F.Cu")
     (at 176.1 132.4 180)
@@
     )
   )
+  (footprint "Button_Switch_SMD:SW_DIP_SPSTx01_Slide_6.7x4.1mm_W6.73mm_P2.54mm_LowProfile_JPin" (layer "F.Cu")
+    (at 210.9724 184.9882)
+    (descr "SMD 1x-dip-switch SPST , Slide, row spacing 6.73 mm (264 mils), body size 6.7x4.1mm (see e.g. https://www.ctscorp.com/wp-content/uploads/219.pdf), SMD, LowProfile, JPin")
+    (tags "SMD DIP Switch SPST Slide 6.73mm 264mil SMD LowProfile JPin")
+    (property "Sheetfile" "Grad_Cap.kicad_sch")
+    (property "Sheetname" "")
+    (attr smd)
+    (fp_text reference "SW1" (at 0 -3.11) (layer "F.SilkS")
+      (effects (font (size 1 1) (thickness 0.15)))
+    )
+    (fp_text value "SW_SPST" (at 0 3.11) (layer "F.Fab")
+      (effects (font (size 1 1) (thickness 0.15)))
+    )
+    (fp_text user "on" (at 0.8975 -1.3425) (layer "F.Fab")
+      (effects (font (size 0.6 0.6) (thickness 0.09)))
+    )
+    (fp_text user "${REFERENCE}" (at 2.58 0 90) (layer "F.Fab")
+      (effects (font (size 0.6 0.6) (thickness 0.09)))
+    )
+    (fp_line (start -1.81 0.565) (end -0.603333 0.565) (layer "F.SilkS") (width 0.12))
+    (fp_line (start -0.603333 -0.635) (end -0.603333 0.635) (layer "F.SilkS") (width 0.12))
+    (fp_line (start -3.65 -2.35) (end -3.65 -0.967) (layer "F.SilkS") (width 0.12))
+    (fp_line (start 3.41 -2.11) (end 3.41 -0.8) (layer "F.SilkS") (width 0.12))
+    (fp_line (start -1.81 0.445) (end -0.603333 0.445) (layer "F.SilkS") (width 0.12))
+    (fp_line (start -1.81 0.635) (end 1.81 0.635) (layer "F.SilkS") (width 0.12))
+    (fp_line (start -3.41 -2.11) (end -3.41 -0.8) (layer "F.SilkS") (width 0.12))
+    (fp_line (start -3.65 -2.35) (end -2.267 -2.35) (layer "F.SilkS") (width 0.12))
+    (fp_line (start -1.81 -0.275) (end -0.603333 -0.275) (layer "F.SilkS") (width 0.12))
+    (fp_line (start -1.81 -0.155) (end -0.603333 -0.155) (layer "F.SilkS") (width 0.12))
+    (fp_line (start -1.81 -0.635) (end -1.81 0.635) (layer "F.SilkS") (width 0.12))
+    (fp_line (start -1.81 0.085) (end -0.603333 0.085) (layer "F.SilkS") (width 0.12))
+    (fp_line (start 1.81 0.635) (end 1.81 -0.635) (layer "F.SilkS") (width 0.12))
+    (fp_line (start -3.41 0.8) (end -3.41 2.11) (layer "F.SilkS") (width 0.12))
+    (fp_line (start 3.41 0.8) (end 3.41 2.11) (layer "F.SilkS") (width 0.12))
+    (fp_line (start -1.81 -0.515) (end -0.603333 -0.515) (layer "F.SilkS") (width 0.12))
+    (fp_line (start -3.41 -2.11) (end 3.41 -2.11) (layer "F.SilkS") (width 0.12))
+    (fp_line (start -1.81 0.325) (end -0.603333 0.325) (layer "F.SilkS") (width 0.12))
+    (fp_line (start -1.81 -0.035) (end -0.603333 -0.035) (layer "F.SilkS") (width 0.12))
+    (fp_line (start -1.81 0.205) (end -0.603333 0.205) (layer "F.SilkS") (width 0.12))
+    (fp_line (start -3.41 2.11) (end 3.41 2.11) (layer "F.SilkS") (width 0.12))
+    (fp_line (start 1.81 -0.635) (end -1.81 -0.635) (layer "F.SilkS") (width 0.12))
+    (fp_line (start -1.81 -0.395) (end -0.603333 -0.395) (layer "F.SilkS") (width 0.12))
+    (fp_line (start -4.7 2.4) (end 4.7 2.4) (layer "F.CrtYd") (width 0.05))
+    (fp_line (start -4.7 -2.4) (end -4.7 2.4) (layer "F.CrtYd") (width 0.05))
+    (fp_line (start 4.7 2.4) (end 4.7 -2.4) (layer "F.CrtYd") (width 0.05))
+    (fp_line (start 4.7 -2.4) (end -4.7 -2.4) (layer "F.CrtYd") (width 0.05))
+    (fp_line (start -1.81 0.565) (end -0.603333 0.565) (layer "F.Fab") (width 0.1))
+    (fp_line (start -1.81 0.165) (end -0.603333 0.165) (layer "F.Fab") (width 0.1))
+    (fp_line (start -3.35 2.05) (end -3.35 -1.05) (layer "F.Fab") (width 0.1))
+    (fp_line (start -1.81 0.065) (end -0.603333 0.065) (layer "F.Fab") (width 0.1))
+    (fp_line (start -1.81 -0.035) (end -0.603333 -0.035) (layer "F.Fab") (width 0.1))
+    (fp_line (start -3.35 -1.05) (end -2.35 -2.05) (layer "F.Fab") (width 0.1))
+    (fp_line (start -1.81 -0.635) (end -1.81 0.635) (layer "F.Fab") (width 0.1))
+    (fp_line (start 3.35 2.05) (end -3.35 2.05) (layer "F.Fab") (width 0.1))
+    (fp_line (start -0.603333 -0.635) (end -0.603333 0.635) (layer "F.Fab") (width 0.1))
+    (fp_line (start -1.81 -0.435) (end -0.603333 -0.435) (layer "F.Fab") (width 0.1))
+    (fp_line (start -1.81 0.465) (end -0.603333 0.465) (layer "F.Fab") (width 0.1))
+    (fp_line (start -1.81 0.635) (end 1.81 0.635) (layer "F.Fab") (width 0.1))
+    (fp_line (start -1.81 0.365) (end -0.603333 0.365) (layer "F.Fab") (width 0.1))
+    (fp_line (start 1.81 -0.635) (end -1.81 -0.635) (layer "F.Fab") (width 0.1))
+    (fp_line (start -1.81 0.265) (end -0.603333 0.265) (layer "F.Fab") (width 0.1))
+    (fp_line (start -2.35 -2.05) (end 3.35 -2.05) (layer "F.Fab") (width 0.1))
+    (fp_line (start -1.81 -0.535) (end -0.603333 -0.535) (layer "F.Fab") (width 0.1))
+    (fp_line (start -1.81 -0.135) (end -0.603333 -0.135) (layer "F.Fab") (width 0.1))
+    (fp_line (start 3.35 -2.05) (end 3.35 2.05) (layer "F.Fab") (width 0.1))
+    (fp_line (start -1.81 -0.235) (end -0.603333 -0.235) (layer "F.Fab") (width 0.1))
+    (fp_line (start 1.81 0.635) (end 1.81 -0.635) (layer "F.Fab") (width 0.1))
+    (fp_line (start -1.81 -0.335) (end -0.603333 -0.335) (layer "F.Fab") (width 0.1))
+    (pad "1" smd rect (at -3.365 0) (size 2.16 1.12) (layers "F.Cu" "F.Paste" "F.Mask")
+      (net 113 "Net-(TP1-Pad1)") (pinfunction "A") (pintype "passive"))
+    (pad "2" smd rect (at 3.365 0) (size 2.16 1.12) (layers "F.Cu" "F.Paste" "F.Mask")
+      (net 2 "+5V") (pinfunction "B") (pintype "passive"))
+    (model "${KICAD6_3DMODEL_DIR}/Button_Switch_SMD.3dshapes/SW_DIP_SPSTx01_Slide_6.7x4.1mm_W6.73mm_P2.54mm_LowProfile_JPin.wrl"
+      (offset (xyz 0 0 0))
+      (scale (xyz 1 1 1))
+      (rotate (xyz 0 0 90))
+    )
+  )
   (footprint "LED_SMD:LED_Inolux_IN-PI554FCH_PLCC4_5.0x5.0mm_P3.2mm" (layer "F.Cu")
     (at 217.329656 165.9636)
@@
     (fp_line (start 2 -2) (end -2 -2) (layer "B.CrtYd") (width 0.05))
     (pad "1" smd rect (at 0 0 180) (size 3 3) (layers "B.Cu" "B.Mask")
-      (net 2 "+5V") (pinfunction "1") (pintype "passive"))
+      (net 113 "Net-(TP1-Pad1)") (pinfunction "1") (pintype "passive"))
   )
   (gr_circle (center 185 185) (end 196.999999 185) (layer "Edge.Cuts") (width 0.1) (fill none))
@@
   (via (at 231.9528 268.1986) (size 0.8) (drill 0.4) (layers "F.Cu" "B.Cu") (net 1))
   (via (at 198.85 201.0344) (size 0.8) (drill 0.4) (layers "F.Cu" "B.Cu") (net 1))
-  (via (at 211.289 185) (size 1.5) (drill 1) (layers "F.Cu" "B.Cu") (net 2))
-  (segment (start 211.289 185) (end 215 185) (width 2.5) (layer "B.Cu") (net 2))
   (segment (start 222.34 244.3478) (end 222.34 247.7921) (width 0.7) (layer "F.Cu") (net 3))
   (segment (start 222.34 247.7921) (end 227.24 252.6921) (width 0.7) (layer "F.Cu") (net 3))
@@
   (segment (start 222.34 221.2592) (end 222.34 223.2798) (width 0.7) (layer "F.Cu") (net 111))
   (segment (start 217.7488 242.8848) (end 219.0142 242.8848) (width 0.7) (layer "F.Cu") (net 112))
+  (segment (start 204.0736 185) (end 207.5956 185) (width 2.5) (layer "F.Cu") (net 113))
+  (segment (start 207.5956 185) (end 207.6074 184.9882) (width 2.5) (layer "F.Cu") (net 113))
+  (via (at 204.0736 185) (size 1.5) (drill 1) (layers "F.Cu" "B.Cu") (net 113))
+  (segment (start 204.0736 185) (end 215 185) (width 2.5) (layer "B.Cu") (net 113))
   (zone (net 2) (net_name "+5V") (layer "F.Cu") (hatch edge 0.508)
     (connect_pads (clearance 0.3))

Commit message: Design has been ordered
Parts:
- removed SW1: SW_SPST, Button_Switch_SMD:SW_DIP_SPSTx01_Slide_6.7x4.1mm_W6.73mm_P2.54mm_LowProfile_JPin
- TP1, TP2: footprint TestPoint:TestPoint_Pad_3.0x3.0mm -> TestPoint:TestPoint_Pad_4.0x4.0mm
- U1: footprint Package_DIP:DIP-28_W16.51mm_SMDSocket_LongPads -> Package_DIP:DIP-28_W15.24mm_LongPads
- moved D5 81.8 mm to (292.0, 225.4), turned to -135 degrees
- moved D6 78.6 mm to (281.7, 235.7), turned to -135 degrees
- moved D7 76.8 mm to (271.4, 245.9), turned to -135 degrees
- moved D8 76.6 mm to (261.1, 256.2), turned to -135 degrees
- moved D4 74.8 mm to (285.1, 218.4), turned to 45 degrees
- moved D28 73.4 mm to (103.1, 210.4), turned to 45 degrees
- moved D29 72.9 mm to (101.1, 199.8), turned to 45 degrees
- moved D27 72.0 mm to (108.6, 219.8), turned to 45 degrees
- moved D26 71.6 mm to (113.8, 228.9), turned to 45 degrees
- moved D30 71.6 mm to (101.2, 188.6), turned to 45 degrees
- moved D31 70.6 mm to (102.3, 178.7), turned to 45 degrees
- moved D25 70.1 mm to (121.8, 237.1), turned to 45 degrees
- moved D9 69.1 mm to (254.2, 249.3), turned to 45 degrees
- moved D32 69.1 mm to (105.1, 168.6), turned to 45 degrees
- moved D3 68.6 mm to (275.6, 219.7), turned to -135 degrees
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Connections:
- TP1 pad 1: Net-(TP1-Pad1) -> +5V
Routing:
- net Net-(TP1-Pad1): track 14.5 -> 0.00 mm, vias 1 -> 0
- net GND: track 172.4 -> 167.1 mm, vias 87 -> 85
- net +5V: track 0.00 -> 4.03 mm, vias 0 -> 1
- net Net-(R1-Pad1): track 15.5 -> 16.2 mm
Other:
- board size 339.4 x 339.4 mm -> 240 x 240 mm
- board text added: "Class of 2023 Bachelor of Science in Mathematics Bachelor of Science in Computer Science"
- board text added: "Designed by Armaan Lala"
