File: Grad_Cap.kicad_sch (KiCad schematic)
At the start: 89 parts, among them U1 ItsyBitsy 32u4 5V

Commit message: Dip Switch
Parts:
- added SW1: SW_SPST, Button_Switch_SMD:SW_DIP_SPSTx01_Slide_6.7x4.1mm_W6.73mm_P2.54mm_LowProfile_JPin, symbol Switch:SW_SPST
Connections:
- net +5V: now also SW1.2 (B); no longer TP1.1
- new net: SW1.1 (A), TP1.1
Other:
- moved on the sheet: TP2
Changed lines of the file:
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@@
     (stroke (width 0) (type default) (color 0 0 0 0))
   )
+  (wire (pts (xy 345.44 78.74) (xy 345.44 77.47))
+    (stroke (width 0) (type default) (color 0 0 0 0))
+  )
   (wire (pts (xy 99.06 44.45) (xy 276.86 44.45))
     (stroke (width 0) (type default) (color 0 0 0 0))
@@
     (stroke (width 0) (type default) (color 0 0 0 0))
   )
+  (wire (pts (xy 335.28 78.74) (xy 335.28 90.17))
+    (stroke (width 0) (type default) (color 0 0 0 0))
+  )
   (wire (pts (xy 193.04 29.21) (xy 196.85 29.21))
     (stroke (width 0) (type default) (color 0 0 0 0))
@@
     (stroke (width 0) (type default) (color 0 0 0 0))
   )
+  (wire (pts (xy 345.44 77.47) (xy 347.98 77.47))
+    (stroke (width 0) (type default) (color 0 0 0 0))
+  )
   (wire (pts (xy 146.05 152.4) (xy 146.05 153.67))
     (stroke (width 0) (type default) (color 0 0 0 0))
@@
     (stroke (width 0) (type default) (color 0 0 0 0))
   )
-  (wire (pts (xy 350.52 92.71) (xy 350.52 95.25))
+  (wire (pts (xy 356.87 88.9) (xy 356.87 91.44))
     (stroke (width 0) (type default) (color 0 0 0 0))
   )
@@
     (stroke (width 0) (type default) (color 0 0 0 0))
   )
+  (wire (pts (xy 335.28 90.17) (xy 341.63 90.17))
+    (stroke (width 0) (type default) (color 0 0 0 0))
+  )
   (wire (pts (xy 165.1 152.4) (xy 165.1 153.67))
     (stroke (width 0) (type default) (color 0 0 0 0))
@@
     (pin "1")
   )
+  (symbol (lib_id "Switch:SW_SPST") (at 340.36 78.74 0) (unit 1)
+    (in_bom yes) (on_board yes) (fields_autoplaced)
+    (property "Reference" "SW1" (id 0) (at 340.36 72.39 0))
+    (property "Value" "SW_SPST" (id 1) (at 340.36 74.93 0))
+    (property "Footprint" "Button_Switch_SMD:SW_DIP_SPSTx01_Slide_6.7x4.1mm_W6.73mm_P2.54mm_LowProfile_JPin" (id 2) (at 340.36 78.74 0)
+      (effects (font (size 1.27 1.27)) hide)
+    )
+    (property "Datasheet" "~" (id 3) (at 340.36 78.74 0)
+      (effects (font (size 1.27 1.27)) hide)
+    )
+    (pin "1")
+    (pin "2")
+  )
   (symbol (lib_id "LED:Inolux_IN-PI554FCH") (at 146.05 194.31 0) (unit 1)
     (in_bom yes) (on_board yes)
@@
     (pin "1")
   )
+  (symbol (lib_id "power:+5V") (at 347.98 77.47 0) (unit 1)
+    (in_bom yes) (on_board yes) (fields_autoplaced)
+    (property "Reference" "#PWR0252" (id 0) (at 347.98 81.28 0)
+      (effects (font (size 1.27 1.27)) hide)
+    )
+    (property "Value" "+5V" (id 1) (at 347.98 72.39 0))
+    (property "Footprint" "" (id 2) (at 347.98 77.47 0)
+      (effects (font (size 1.27 1.27)) hide)
+    )
+    (property "Datasheet" "" (id 3) (at 347.98 77.47 0)
+      (effects (font (size 1.27 1.27)) hide)
+    )
+    (pin "1")
+  )
   (symbol (lib_id "LED:Inolux_IN-PI554FCH") (at 224.79 161.29 0) (unit 1)
     (in_bom yes) (on_board yes)
@@
     (pin "1")
   )
-  (symbol (lib_id "power:+5V") (at 341.63 90.17 0) (unit 1)
-    (in_bom yes) (on_board yes) (fields_autoplaced)
-    (property "Reference" "#PWR0252" (id 0) (at 341.63 93.98 0)
-      (effects (font (size 1.27 1.27)) hide)
-    )
-    (property "Value" "+5V" (id 1) (at 341.63 85.09 0))
-    (property "Footprint" "" (id 2) (at 341.63 90.17 0)
-      (effects (font (size 1.27 1.27)) hide)
-    )
-    (property "Datasheet" "" (id 3) (at 341.63 90.17 0)
-      (effects (font (size 1.27 1.27)) hide)
-    )
-    (pin "1")
-  )
   (symbol (lib_id "power:+5V") (at 264.16 218.44 0) (unit 1)
     (in_bom yes) (on_board yes) (fields_autoplaced)
@@
     (pin "4")
   )
-  (symbol (lib_name "GND_3") (lib_id "power:GND") (at 350.52 95.25 0) (unit 1)
+  (symbol (lib_name "GND_3") (lib_id "power:GND") (at 356.87 91.44 0) (unit 1)
     (in_bom yes) (on_board yes) (fields_autoplaced)
-    (property "Reference" "#PWR0258" (id 0) (at 350.52 101.6 0)
+    (property "Reference" "#PWR0258" (id 0) (at 356.87 97.79 0)
       (effects (font (size 1.27 1.27)) hide)
     )
-    (property "Value" "GND" (id 1) (at 350.52 100.33 0))
-    (property "Footprint" "" (id 2) (at 350.52 95.25 0)
+    (property "Value" "GND" (id 1) (at 356.87 96.52 0))
+    (property "Footprint" "" (id 2) (at 356.87 91.44 0)
       (effects (font (size 1.27 1.27)) hide)
     )
-    (property "Datasheet" "" (id 3) (at 350.52 95.25 0)
+    (property "Datasheet" "" (id 3) (at 356.87 91.44 0)
       (effects (font (size 1.27 1.27)) hide)
     )
@@
     (pin "1")
   )
-  (symbol (lib_id "Connector:TestPoint") (at 350.52 92.71 0) (unit 1)
+  (symbol (lib_id "Connector:TestPoint") (at 356.87 88.9 0) (unit 1)
     (in_bom yes) (on_board yes) (fields_autoplaced)
-    (property "Reference" "TP2" (id 0) (at 353.06 88.1379 0)
+    (property "Reference" "TP2" (id 0) (at 359.41 84.3279 0)
       (effects (font (size 1.27 1.27)) (justify left))
     )
-    (property "Value" "TestPoint" (id 1) (at 353.06 90.6779 0)
+    (property "Value" "TestPoint" (id 1) (at 359.41 86.8679 0)
       (effects (font (size 1.27 1.27)) (justify left))
     )
-    (property "Footprint" "TestPoint:TestPoint_Pad_4.0x4.0mm" (id 2) (at 355.6 92.71 0)
+    (property "Footprint" "TestPoint:TestPoint_Pad_4.0x4.0mm" (id 2) (at 361.95 88.9 0)
       (effects (font (size 1.27 1.27)) hide)
     )
-    (property "Datasheet" "" (id 3) (at 355.6 92.71 0)
+    (property "Datasheet" "" (id 3) (at 361.95 88.9 0)
       (effects (font (size 1.27 1.27)) hide)
     )
@@
       (reference "#PWR0251") (unit 1) (value "GND") (footprint "")
     )
-    (path "/6e3dc5c3-5494-438e-85ba-85658666f454"
+    (path "/4d155719-0793-4183-8ab5-1f8f63d620d8"
       (reference "#PWR0252") (unit 1) (value "+5V") (footprint "")
     )
@@
       (reference "R1") (unit 1) (value "330") (footprint "Resistor_SMD:R_1206_3216Metric_Pad1.30x1.75mm_HandSolder")
     )
+    (path "/1cf5988c-c21e-4031-b577-f3f4d2070ea1"
+      (reference "SW1") (unit 1) (value "SW_SPST") (footprint "Button_Switch_SMD:SW_DIP_SPSTx01_Slide_6.7x4.1mm_W6.73mm_P2.54mm_LowProfile_JPin")
+    )
     (path "/9dde1d2c-cc43-4a60-a255-4b69425034cd"

Commit message: Design has been ordered
Parts:
- removed SW1: SW_SPST, Button_Switch_SMD:SW_DIP_SPSTx01_Slide_6.7x4.1mm_W6.73mm_P2.54mm_LowProfile_JPin, symbol Switch:SW_SPST
Connections:
- net +5V: now also TP1.1
Changed lines of the file:
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@@
     (stroke (width 0) (type default) (color 0 0 0 0))
   )
-  (wire (pts (xy 345.44 78.74) (xy 345.44 77.47))
-    (stroke (width 0) (type default) (color 0 0 0 0))
-  )
   (wire (pts (xy 99.06 44.45) (xy 276.86 44.45))
     (stroke (width 0) (type default) (color 0 0 0 0))
@@
     (stroke (width 0) (type default) (color 0 0 0 0))
   )
-  (wire (pts (xy 335.28 78.74) (xy 335.28 90.17))
-    (stroke (width 0) (type default) (color 0 0 0 0))
-  )
   (wire (pts (xy 193.04 29.21) (xy 196.85 29.21))
     (stroke (width 0) (type default) (color 0 0 0 0))
@@
     (stroke (width 0) (type default) (color 0 0 0 0))
   )
-  (wire (pts (xy 106.68 168.91) (xy 106.68 170.18))
-    (stroke (width 0) (type default) (color 0 0 0 0))
-  )
   (wire (pts (xy 153.67 194.31) (xy 157.48 194.31))
     (stroke (width 0) (type default) (color 0 0 0 0))
@@
     (stroke (width 0) (type default) (color 0 0 0 0))
   )
-  (wire (pts (xy 106.68 152.4) (xy 106.68 153.67))
-    (stroke (width 0) (type default) (color 0 0 0 0))
-  )
   (wire (pts (xy 99.06 242.57) (xy 276.86 242.57))
     (stroke (width 0) (type default) (color 0 0 0 0))
@@
     (stroke (width 0) (type default) (color 0 0 0 0))
   )
-  (wire (pts (xy 341.63 90.17) (xy 341.63 92.71))
-    (stroke (width 0) (type default) (color 0 0 0 0))
-  )
   (wire (pts (xy 153.67 260.35) (xy 157.48 260.35))
     (stroke (width 0) (type default) (color 0 0 0 0))
@@
     (stroke (width 0) (type default) (color 0 0 0 0))
   )
-  (wire (pts (xy 345.44 77.47) (xy 347.98 77.47))
-    (stroke (width 0) (type default) (color 0 0 0 0))
-  )
   (wire (pts (xy 146.05 152.4) (xy 146.05 153.67))
     (stroke (width 0) (type default) (color 0 0 0 0))
@@
     (stroke (width 0) (type default) (color 0 0 0 0))
   )
-  (wire (pts (xy 341.63 146.05) (xy 341.63 140.97))
-    (stroke (width 0) (type default) (color 0 0 0 0))
-  )
   (wire (pts (xy 264.16 152.4) (xy 264.16 153.67))
     (stroke (width 0) (type default) (color 0 0 0 0))
@@
     (stroke (width 0) (type default) (color 0 0 0 0))
   )
+  (wire (pts (xy 341.63 85.09) (xy 341.63 92.71))
+    (stroke (width 0) (type default) (color 0 0 0 0))
+  )
   (wire (pts (xy 165.1 234.95) (xy 165.1 236.22))
     (stroke (width 0) (type default) (color 0 0 0 0))
@@
     (stroke (width 0) (type default) (color 0 0 0 0))
   )
-  (wire (pts (xy 335.28 90.17) (xy 341.63 90.17))
-    (stroke (width 0) (type default) (color 0 0 0 0))
-  )
   (wire (pts (xy 165.1 152.4) (xy 165.1 153.67))
     (stroke (width 0) (type default) (color 0 0 0 0))
@@
     (pin "1")
   )
-  (symbol (lib_id "Switch:SW_SPST") (at 340.36 78.74 0) (unit 1)
-    (in_bom yes) (on_board yes) (fields_autoplaced)
-    (property "Reference" "SW1" (id 0) (at 340.36 72.39 0))
-    (property "Value" "SW_SPST" (id 1) (at 340.36 74.93 0))
-    (property "Footprint" "Button_Switch_SMD:SW_DIP_SPSTx01_Slide_6.7x4.1mm_W6.73mm_P2.54mm_LowProfile_JPin" (id 2) (at 340.36 78.74 0)
-      (effects (font (size 1.27 1.27)) hide)
-    )
-    (property "Datasheet" "~" (id 3) (at 340.36 78.74 0)
-      (effects (font (size 1.27 1.27)) hide)
-    )
-    (pin "1")
-    (pin "2")
-  )
   (symbol (lib_id "LED:Inolux_IN-PI554FCH") (at 146.05 194.31 0) (unit 1)
     (in_bom yes) (on_board yes)
@@
     (pin "1")
   )
-  (symbol (lib_id "power:+5V") (at 347.98 77.47 0) (unit 1)
+  (symbol (lib_id "power:+5V") (at 341.63 85.09 0) (unit 1)
     (in_bom yes) (on_board yes) (fields_autoplaced)
-    (property "Reference" "#PWR0252" (id 0) (at 347.98 81.28 0)
+    (property "Reference" "#PWR0252" (id 0) (at 341.63 88.9 0)
       (effects (font (size 1.27 1.27)) hide)
     )
-    (property "Value" "+5V" (id 1) (at 347.98 72.39 0))
-    (property "Footprint" "" (id 2) (at 347.98 77.47 0)
+    (property "Value" "+5V" (id 1) (at 341.63 80.01 0))
+    (property "Footprint" "" (id 2) (at 341.63 85.09 0)
       (effects (font (size 1.27 1.27)) hide)
     )
-    (property "Datasheet" "" (id 3) (at 347.98 77.47 0)
+    (property "Datasheet" "" (id 3) (at 341.63 85.09 0)
       (effects (font (size 1.27 1.27)) hide)
     )
@@
     (pin "1")
   )
-  (symbol (lib_id "power:+5V") (at 106.68 152.4 0) (unit 1)
-    (in_bom yes) (on_board yes) (fields_autoplaced)
-    (property "Reference" "#PWR0230" (id 0) (at 106.68 156.21 0)
-      (effects (font (size 1.27 1.27)) hide)
-    )
-    (property "Value" "+5V" (id 1) (at 106.68 147.32 0))
-    (property "Footprint" "" (id 2) (at 106.68 152.4 0)
-      (effects (font (size 1.27 1.27)) hide)
-    )
-    (property "Datasheet" "" (id 3) (at 106.68 152.4 0)
-      (effects (font (size 1.27 1.27)) hide)
-    )
-    (pin "1")
-  )
   (symbol (lib_id "LED:Inolux_IN-PI554FCH") (at 127 128.27 0) (unit 1)
     (in_bom yes) (on_board yes)
@@
     (pin "1")
   )
-  (symbol (lib_id "power:GND") (at 106.68 170.18 0) (unit 1)
-    (in_bom yes) (on_board yes) (fields_autoplaced)
-    (property "Reference" "#PWR0239" (id 0) (at 106.68 176.53 0)
-      (effects (font (size 1.27 1.27)) hide)
-    )
-    (property "Value" "GND" (id 1) (at 106.68 175.26 0))
-    (property "Footprint" "" (id 2) (at 106.68 170.18 0)
-      (effects (font (size 1.27 1.27)) hide)
-    )
-    (property "Datasheet" "" (id 3) (at 106.68 170.18 0)
-      (effects (font (size 1.27 1.27)) hide)
-    )
-    (pin "1")
-  )
   (symbol (lib_id "power:GND") (at 317.5 191.77 90) (unit 1)
     (in_bom yes) (on_board yes) (fields_autoplaced)
@@
       (reference "#PWR0229") (unit 1) (value "+5V") (footprint "")
     )
-    (path "/8dc9667b-9115-4571-9f7f-91ad6103712a"
-      (reference "#PWR0230") (unit 1) (value "+5V") (footprint "")
-    )
     (path "/f98ab731-1f3a-4f42-9208-7517ecca2e12"
       (reference "#PWR0231") (unit 1) (value "+5V") (footprint "")
@@
       (reference "#PWR0238") (unit 1) (value "+5V") (footprint "")
     )
-    (path "/ce8416b5-92aa-4e19-a088-e3d5a53076d1"
-      (reference "#PWR0239") (unit 1) (value "GND") (footprint "")
-    )
     (path "/6030ea99-9fb6-4573-8909-d0103fcee3bf"
       (reference "#PWR0240") (unit 1) (value "+5V") (footprint "")
@@
       (reference "R1") (unit 1) (value "330") (footprint "Resistor_SMD:R_1206_3216Metric_Pad1.30x1.75mm_HandSolder")
     )
-    (path "/1cf5988c-c21e-4031-b577-f3f4d2070ea1"
-      (reference "SW1") (unit 1) (value "SW_SPST") (footprint "Button_Switch_SMD:SW_DIP_SPSTx01_Slide_6.7x4.1mm_W6.73mm_P2.54mm_LowProfile_JPin")
-    )
     (path "/9dde1d2c-cc43-4a60-a255-4b69425034cd"
